File: throwie/hardware/RevB/throwie/throwie.kicad_pcb (KiCad board)
At the start: 2 copper layers, 33.8 x 18.8 mm, 24 parts, among them J1 CONN, Q1 2SC3356, Q2 SS8050-G, T1 TestPoints, T2 TestPoints, T3 TestPoints, T4 TestPoints, U1 C8051F850-A-GU, U2 MIC5231-3.3YM5-TR, X1 RO3101

Commit message: drill file
Routing:
- net +BATT: track 43.2 -> 40.1 mm, vias 3 -> 2
Changed lines of the file:
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@@
     (thickness 1.6)
     (drawings 33)
-    (tracks 275)
+    (tracks 272)
     (zones 0)
     (modules 24)
@@
   )
   (setup
-    (last_trace_width 1)
+    (last_trace_width 0.5)
     (user_trace_width 0.4)
     (user_trace_width 0.5)
@@
   (segment (start 45.108 161.036) (end 39.878 161.036) (width 1) (layer B.Cu) (net 3))
   (segment (start 35.258 161.036) (end 39.878 161.036) (width 1.5) (layer F.Cu) (net 3))
-  (via (at 42.164 157.48) (size 0.8) (drill 0.4) (layers F.Cu B.Cu) (net 3))
   (via (at 41.148 157.48) (size 0.8) (drill 0.4) (layers F.Cu B.Cu) (net 3))
   (segment (start 39.861823 161.08364) (end 39.861823 159.782177) (width 1) (layer F.Cu) (net 3))
@@
   (segment (start 39.878 158.75) (end 42.164 156.464) (width 1) (layer F.Cu) (net 3))
   (segment (start 39.878 159.766) (end 39.878 158.75) (width 1) (layer F.Cu) (net 3))
-  (segment (start 42.164 156.914315) (end 42.164 157.48) (width 0.5) (layer B.Cu) (net 3))
-  (segment (start 42.164 155.898315) (end 42.164 156.914315) (width 0.5) (layer B.Cu) (net 3))
-  (segment (start 44.900315 153.162) (end 42.164 155.898315) (width 0.5) (layer B.Cu) (net 3))
-  (segment (start 47.073 153.162) (end 44.900315 153.162) (width 0.5) (layer B.Cu) (net 3))
   (segment (start 47.835 153.924) (end 47.073 153.162) (width 0.5) (layer B.Cu) (net 3))
   (segment (start 41.148 157.48) (end 42.164 156.464) (width 1) (layer B.Cu) (net 3))
-  (segment (start 41.148 157.48) (end 42.164 157.48) (width 1) (layer B.Cu) (net 3))
-  (segment (start 42.164 156.464) (end 42.164 157.48) (width 1) (layer B.Cu) (net 3))
+  (segment (start 43.79999 154.82801) (end 43.79999 154.32001) (width 0.5) (layer B.Cu) (net 3))
+  (segment (start 42.164 156.464) (end 43.79999 154.82801) (width 0.5) (layer B.Cu) (net 3))
+  (segment (start 44.958 153.162) (end 47.073 153.162) (width 0.5) (layer B.Cu) (net 3))
+  (segment (start 43.79999 154.32001) (end 44.958 153.162) (width 0.5) (layer B.Cu) (net 3))
   (segment (start 49.276 154.559) (end 51.943 154.559) (width 0.4) (layer F.Cu) (net 4))
   (segment (start 51.943 154.559) (end 52.07 154.432) (width 0.4) (layer F.Cu) (net 4))
